Commit message: fixed positions

File: body.urdf (robot description, URDF)
Before this commit: robot robot, 2 links, 1 joints
Joints:
- joint Link0_Link1: origin xyz=0.5 0 1 rpy=0 0 0 -> xyz=0 0 1 rpy=0 0 0

Commit message: link 4

File: body.urdf (robot description, URDF)
Before this commit: robot robot, 3 links, 2 joints
Links:
- added link Link3, mass 1; collision box size=1 1 1; visual box size=1 1 1
- added link Link4, mass 1; collision box size=1 1 1; visual box size=1 1 1
Joints:
- added joint Link2_Link3: type revolute, parent Link2, child Link3, origin xyz=0 0.5 0.5 rpy=0 0 0, axis 0 1 0, limit lower=-3.14159 upper=3.14159 effort=0.0 velocity=0.0
- added joint Link3_Link4: type revolute, parent Link3, child Link4, origin xyz=0 1 0 rpy=0 0 0, axis 0 1 0, limit lower=-3.14159 upper=3.14159 effort=0.0 velocity=0.0

Commit message: added link 5

File: body.urdf (robot description, URDF)
Before this commit: robot robot, 5 links, 4 joints
Links:
- added link Link5, mass 1; collision box size=1 1 1; visual box size=1 1 1
Joints:
- added joint Link4_Link5: type revolute, parent Link4, child Link5, origin xyz=0 0.5 -0.5 rpy=0 0 0, axis 0 1 0, limit lower=-3.14159 upper=3.14159 effort=0.0 velocity=0.0

Commit message: front leg size

File: body.urdf (robot description, URDF)
Before this commit: robot robot, 3 links, 2 joints
Links:
- link FrontLeg: geometry collision box size=0.2 1 0.2; visual box size=0.2 1 0.2

Commit message: torso backleg

File: body.urdf (robot description, URDF)
Before this commit: robot robot, 3 links, 2 joints
Joints:
- joint Torso_BackLeg: origin xyz=1 0 1 rpy=0 0 0 -> xyz=0 -0.5 1 rpy=0 0 0

Commit message: backleg

File: body.urdf (robot description, URDF)
Before this commit: robot robot, 3 links, 2 joints
Links:
- link BackLeg: geometry collision box size=0.2 1 0.2; visual box size=0.2 1 0.2

Commit message: frontlower

File: body.urdf (robot description, URDF)
Before this commit: robot robot, 5 links, 4 joints
Links:
- added link FrontLowerLeg, mass 1; collision box size=0.2 0.2 1; visual box size=0.2 0.2 1
Joints:
- added joint FrontLeg_FrontLowerLeg: type revolute, parent FrontLeg, child FrontLowerLeg, origin xyz=0 1 0 rpy=0 0 0, axis 1 0 0, limit lower=-3.14159 upper=3.14159 effort=0.0 velocity=0.0

Commit message: backlower

File: body.urdf (robot description, URDF)
Before this commit: robot robot, 6 links, 5 joints
Links:
- added link BackLowerLeg, mass 1; collision box size=0.2 0.2 1; visual box size=0.2 0.2 1
Joints:
- added joint BackLeg_BackLowerLeg: type revolute, parent BackLeg, child BackLowerLeg, origin xyz=0 -1 0 rpy=0 0 0, axis 1 0 0, limit lower=-3.14159 upper=3.14159 effort=0.0 velocity=0.0

Commit message: leftlower

File: body.urdf (robot description, URDF)
Before this commit: robot robot, 7 links, 6 joints
Links:
- added link LeftLowerLeg, mass 1; collision box size=0.2 0.2 1; visual box size=0.2 0.2 1
Joints:
- added joint LeftLeg_LeftLowerLeg: type revolute, parent LeftLeg, child LeftLowerLeg, origin xyz=-1 0 0 rpy=0 0 0, axis 0 1 0, limit lower=-3.14159 upper=3.14159 effort=0.0 velocity=0.0

Commit message: rightlower

File: body.urdf (robot description, URDF)
Before this commit: robot robot, 8 links, 7 joints
Links:
- added link RightLowerLeg, mass 1; collision box size=0.2 0.2 1; visual box size=0.2 0.2 1
Joints:
- added joint RightLeg_RightLowerLeg: type revolute, parent RightLeg, child RightLowerLeg, origin xyz=1 0 0 rpy=0 0 0, axis 0 1 0, limit lower=-3.14159 upper=3.14159 effort=0.0 velocity=0.0

Commit message: added back foot

File: body.urdf (robot description, URDF)
Before this commit: robot robot, 9 links, 8 joints
Links:
- added link BackFoot, mass 1; collision box size=0.75 0.75 0.2; visual box size=0.75 0.75 0.2
Joints:
- added joint BackLowerLeg_BackFoot: type revolute, parent BackLowerLeg, child BackFoot, origin xyz=0 0 -1 rpy=0 0 0, axis 1 0 0, limit lower=-3.14159 upper=3.14159 effort=0.0 velocity=0.0

Commit message: added front foot

File: body.urdf (robot description, URDF)
Before this commit: robot robot, 10 links, 9 joints
Links:
- added link FrontFoot, mass 1; collision box size=0.75 0.75 0.2; visual box size=0.75 0.75 0.2
Joints:
- added joint FrontLowerLeg_FrontFoot: type revolute, parent FrontLowerLeg, child FrontFoot, origin xyz=0 0 -1 rpy=0 0 0, axis 1 0 0, limit lower=-3.14159 upper=3.14159 effort=0.0 velocity=0.0

Commit message: added left foot

File: body.urdf (robot description, URDF)
Before this commit: robot robot, 11 links, 10 joints
Links:
- added link LeftFoot, mass 1; collision box size=0.75 0.75 0.2; visual box size=0.75 0.75 0.2
Joints:
- added joint LeftLowerLeg_LeftFoot: type revolute, parent LeftLowerLeg, child LeftFoot, origin xyz=0 0 -1 rpy=0 0 0, axis 0 1 0, limit lower=-3.14159 upper=3.14159 effort=0.0 velocity=0.0

Commit message: added right foot

File: body.urdf (robot description, URDF)
Before this commit: robot robot, 12 links, 11 joints
Links:
- added link RightFoot, mass 1; collision box size=0.75 0.75 0.2; visual box size=0.75 0.75 0.2
Joints:
- added joint RightLowerLeg_RightFoot: type revolute, parent RightLowerLeg, child RightFoot, origin xyz=0 0 -1 rpy=0 0 0, axis 0 1 0, limit lower=-3.14159 upper=3.14159 effort=0.0 velocity=0.0
- joint Torso_BackLeg: origin xyz=0 -0.5 1 rpy=0 0 0 -> xyz=0 -0.5 1.5 rpy=0 0 0
- joint Torso_FrontLeg: origin xyz=0 0.5 1 rpy=0 0 0 -> xyz=0 0.5 1.5 rpy=0 0 0
- joint Torso_LeftLeg: origin xyz=-0.5 0 1 rpy=0 0 0 -> xyz=-0.5 0 1.5 rpy=0 0 0
- joint Torso_RightLeg: origin xyz=0.5 0 1 rpy=0 0 0 -> xyz=0.5 0 1.5 rpy=0 0 0

Commit message: done feet

File: body.urdf (robot description, URDF)
Before this commit: robot robot, 13 links, 12 joints
Joints:
- joint Torso_BackLeg: origin xyz=0 -0.5 1.5 rpy=0 0 0 -> xyz=0 -0.5 1.2 rpy=0 0 0
- joint Torso_FrontLeg: origin xyz=0 0.5 1.5 rpy=0 0 0 -> xyz=0 0.5 1.2 rpy=0 0 0
- joint Torso_LeftLeg: origin xyz=-0.5 0 1.5 rpy=0 0 0 -> xyz=-0.5 0 1.2 rpy=0 0 0
- joint Torso_RightLeg: origin xyz=0.5 0 1.5 rpy=0 0 0 -> xyz=0.5 0 1.2 rpy=0 0 0

Commit message: rightback

File: body.urdf (robot description, URDF)
Before this commit: robot robot, 13 links, 12 joints
Links:
- removed link BackFoot
- removed link BackLeg
- removed link BackLowerLeg
- removed link FrontFoot
- removed link FrontLeg
- removed link FrontLowerLeg
- removed link LeftFoot
- removed link LeftLeg
- removed link LeftLowerLeg
- removed link RightFoot
- removed link RightLeg
- removed link RightLowerLeg
- added link RightBack, mass 1; collision box size=0.2 0.2 0.5; visual box size=0.2 0.2 0.5
- link Torso: geometry collision box size=1 2 1; visual box size=1 2 1
Joints:
- removed joint BackLeg_BackLowerLeg
- removed joint BackLowerLeg_BackFoot
- removed joint FrontLeg_FrontLowerLeg
- removed joint FrontLowerLeg_FrontFoot
- removed joint LeftLeg_LeftLowerLeg
- removed joint LeftLowerLeg_LeftFoot
- removed joint RightLeg_RightLowerLeg
- removed joint RightLowerLeg_RightFoot
- removed joint Torso_BackLeg
- removed joint Torso_FrontLeg
- removed joint Torso_LeftLeg
- removed joint Torso_RightLeg
- added joint Torso_RightBack: type revolute, parent Torso, child RightBack, origin xyz=-0.25 -0.5 0.7 rpy=0 0 0, axis 0 1 0, limit lower=-3.14159 upper=3.14159 effort=0.0 velocity=0.0

Commit message: rightfront

File: body.urdf (robot description, URDF)
Before this commit: robot robot, 2 links, 1 joints
Links:
- added link RightFront, mass 1; collision box size=0.2 0.2 0.5; visual box size=0.2 0.2 0.5
Joints:
- added joint Torso_RightFront: type revolute, parent Torso, child RightFront, origin xyz=0.25 -0.5 0.7 rpy=0 0 0, axis 0 1 0, limit lower=-3.14159 upper=3.14159 effort=0.0 velocity=0.0

Commit message: fixed height

File: body.urdf (robot description, URDF)
Before this commit: robot robot, 3 links, 2 joints
Links:
- added link LeftBack, mass 1; collision box size=0.2 0.2 0.5; visual box size=0.2 0.2 0.5
- link Torso: geometry collision box size=1 2 0.5; visual box size=1 2 0.5
Joints:
- added joint Torso_LeftBack: type revolute, parent Torso, child LeftBack, origin xyz=-0.25 0.5 0.95 rpy=0 0 0, axis 0 1 0, limit lower=-3.14159 upper=3.14159 effort=0.0 velocity=0.0
- joint Torso_RightBack: origin xyz=-0.25 -0.5 0.7 rpy=0 0 0 -> xyz=-0.25 -0.5 0.95 rpy=0 0 0
- joint Torso_RightFront: origin xyz=0.25 -0.5 0.7 rpy=0 0 0 -> xyz=0.25 -0.5 0.95 rpy=0 0 0

Commit message: leftfront

File: body.urdf (robot description, URDF)
Before this commit: robot robot, 4 links, 3 joints
Links:
- added link LeftFront, mass 1; collision box size=0.2 0.2 0.5; visual box size=0.2 0.2 0.5
Joints:
- added joint Torso_LeftFront: type revolute, parent Torso, child LeftFront, origin xyz=0.25 0.5 0.95 rpy=0 0 0, axis 0 1 0, limit lower=-3.14159 upper=3.14159 effort=0.0 velocity=0.0

Commit message: rightlowerback

File: body.urdf (robot description, URDF)
Before this commit: robot robot, 5 links, 4 joints
Links:
- added link LowerRB, mass 1; collision box size=0.2 0.2 0.5; visual box size=0.2 0.2 0.5
Joints:
- added joint RightBack_LowerRB: type revolute, parent RightBack, child LowerRB, origin xyz=0 0 -0.5 rpy=0 0 0, axis 0 1 0, limit lower=-3.14159 upper=3.14159 effort=0.0 velocity=0.0

Commit message: put box

File: body.urdf (robot description, URDF)
Before this commit: robot robot, 13 links, 12 joints
Links:
- removed link BackFoot
- removed link BackLeg
- removed link BackLowerLeg
- removed link FrontFoot
- removed link FrontLeg
- removed link FrontLowerLeg
- removed link LeftFoot
- removed link LeftLeg
- removed link LeftLowerLeg
- removed link RightFoot
- removed link RightLeg
- removed link RightLowerLeg
- link Torso: geometry collision box size=1 0.5 0.5; visual box size=1 0.5 0.5
Joints:
- removed joint BackLeg_BackLowerLeg
- removed joint BackLowerLeg_BackFoot
- removed joint FrontLeg_FrontLowerLeg
- removed joint FrontLowerLeg_FrontFoot
- removed joint LeftLeg_LeftLowerLeg
- removed joint LeftLowerLeg_LeftFoot
- removed joint RightLeg_RightLowerLeg
- removed joint RightLowerLeg_RightFoot
- removed joint Torso_BackLeg
- removed joint Torso_FrontLeg
- removed joint Torso_LeftLeg
- removed joint Torso_RightLeg

Commit message: added frontleft

File: body.urdf (robot description, URDF)
Before this commit: robot robot, 1 links, 0 joints
Links:
- added link FrontLeft, mass 1; collision box size=0.2 0.5 0.2; visual box size=0.2 0.5 0.2
Joints:
- added joint Torso_FrontLeft: type revolute, parent Torso, child FrontLeft, origin xyz=0.25 0.25 1 rpy=0 0 0, axis 1 0 0, limit lower=-3.14159 upper=3.14159 effort=0.0 velocity=0.0

Commit message: added frontright

File: body.urdf (robot description, URDF)
Before this commit: robot robot, 2 links, 1 joints
Links:
- added link FrontRight, mass 1; collision box size=0.2 0.5 0.2; visual box size=0.2 0.5 0.2
Joints:
- added joint Torso_FrontRight: type revolute, parent Torso, child FrontRight, origin xyz=-0.25 0.25 1 rpy=0 0 0, axis 1 0 0, limit lower=-3.14159 upper=3.14159 effort=0.0 velocity=0.0

Commit message: added backleft

File: body.urdf (robot description, URDF)
Before this commit: robot robot, 3 links, 2 joints
Links:
- removed link FrontRight
- added link BackLeft, mass 1; collision box size=0.2 0.5 0.2; visual box size=0.2 0.5 0.2
Joints:
- removed joint Torso_FrontRight
- added joint Torso_BackLeft: type revolute, parent Torso, child BackLeft, origin xyz=0.25 -0.25 1 rpy=0 0 0, axis 1 0 0, limit lower=-3.14159 upper=3.14159 effort=0.0 velocity=0.0

Commit message: FLLower

File: body.urdf (robot description, URDF)
Before this commit: robot robot, 3 links, 2 joints
Links:
- added link BackRight, mass 1; collision box size=0.2 0.5 0.2; visual box size=0.2 0.5 0.2
- added link FLLower, mass 1; collision box size=0.2 0.2 0.5; visual box size=0.2 0.2 0.5
- added link FrontRight, mass 1; collision box size=0.2 0.5 0.2; visual box size=0.2 0.5 0.2
Joints:
- added joint FrontLeft_FLLower: type revolute, parent FrontLeft, child FLLower, origin xyz=0 0.5 0 rpy=0 0 0, axis 1 0 0, limit lower=-3.14159 upper=3.14159 effort=0.0 velocity=0.0
- added joint Torso_BackRight: type revolute, parent Torso, child BackRight, origin xyz=0.25 -0.25 1 rpy=0 0 0, axis 1 0 0, limit lower=-3.14159 upper=3.14159 effort=0.0 velocity=0.0
- added joint Torso_FrontRight: type revolute, parent Torso, child FrontRight, origin xyz=0.25 0.25 1 rpy=0 0 0, axis 1 0 0, limit lower=-3.14159 upper=3.14159 effort=0.0 velocity=0.0
- joint Torso_BackLeft: origin xyz=0.25 -0.25 1 rpy=0 0 0 -> xyz=-0.25 -0.25 1 rpy=0 0 0
- joint Torso_FrontLeft: origin xyz=0.25 0.25 1 rpy=0 0 0 -> xyz=-0.25 0.25 1 rpy=0 0 0

Commit message: FR and BL lower

File: body.urdf (robot description, URDF)
Before this commit: robot robot, 6 links, 5 joints
Links:
- added link FRLower, mass 1; collision box size=0.2 0.2 0.5; visual box size=0.2 0.2 0.5
Joints:
- added joint FrontRight_FRLower: type revolute, parent FrontRight, child FRLower, origin xyz=0 0.5 0 rpy=0 0 0, axis 1 0 0, limit lower=-3.14159 upper=3.14159 effort=0.0 velocity=0.0

Commit message: BRLower

File: body.urdf (robot description, URDF)
Before this commit: robot robot, 7 links, 6 joints
Links:
- added link BLLower, mass 1; collision box size=0.2 0.2 0.5; visual box size=0.2 0.2 0.5
- added link BRLower, mass 1; collision box size=0.2 0.2 0.5; visual box size=0.2 0.2 0.5
Joints:
- added joint BackLeft_BLLower: type revolute, parent BackLeft, child BLLower, origin xyz=0 -0.5 0 rpy=0 0 0, axis 1 0 0, limit lower=-3.14159 upper=3.14159 effort=0.0 velocity=0.0
- added joint BackRight_BRLower: type revolute, parent BackRight, child BRLower, origin xyz=0 -0.5 0 rpy=0 0 0, axis 1 0 0, limit lower=-3.14159 upper=3.14159 effort=0.0 velocity=0.0

Commit message: fixed leglength

File: body.urdf (robot description, URDF)
Before this commit: robot robot, 9 links, 8 joints
Links:
- link BLLower: geometry collision box size=0.2 0.2 0.75; visual box size=0.2 0.2 0.75
- link BRLower: geometry collision box size=0.2 0.2 0.75; visual box size=0.2 0.2 0.75
- link BackLeft: geometry collision box size=0.2 0.75 0.2; visual box size=0.2 0.75 0.2
- link BackRight: geometry collision box size=0.2 0.75 0.2; visual box size=0.2 0.75 0.2
- link FLLower: geometry collision box size=0.2 0.2 0.75; visual box size=0.2 0.2 0.75
- link FRLower: geometry collision box size=0.2 0.2 0.75; visual box size=0.2 0.2 0.75
- link FrontLeft: geometry collision box size=0.2 0.75 0.2; visual box size=0.2 0.75 0.2
- link FrontRight: geometry collision box size=0.2 0.75 0.2; visual box size=0.2 0.75 0.2
Joints:
- joint BackLeft_BLLower: origin xyz=0 -0.5 0 rpy=0 0 0 -> xyz=0 -0.75 0 rpy=0 0 0
- joint BackRight_BRLower: origin xyz=0 -0.5 0 rpy=0 0 0 -> xyz=0 -0.75 0 rpy=0 0 0
- joint FrontLeft_FLLower: origin xyz=0 0.5 0 rpy=0 0 0 -> xyz=0 0.75 0 rpy=0 0 0
- joint FrontRight_FRLower: origin xyz=0 0.5 0 rpy=0 0 0 -> xyz=0 0.75 0 rpy=0 0 0
- joint Torso_BackLeft: origin xyz=-0.25 -0.25 1 rpy=0 0 0 -> xyz=-0.25 -0.25 0.75 rpy=0 0 0
- joint Torso_BackRight: origin xyz=0.25 -0.25 1 rpy=0 0 0 -> xyz=0.25 -0.25 0.75 rpy=0 0 0
- joint Torso_FrontLeft: origin xyz=-0.25 0.25 1 rpy=0 0 0 -> xyz=-0.25 0.25 0.75 rpy=0 0 0
- joint Torso_FrontRight: origin xyz=0.25 0.25 1 rpy=0 0 0 -> xyz=0.25 0.25 0.75 rpy=0 0 0

Commit message: added side legs

File: body.urdf (robot description, URDF)
Before this commit: robot robot, 9 links, 8 joints
Links:
- added link Left, mass 1; collision box size=0.75 0.2 0.2; visual box size=0.75 0.2 0.2
- added link LeftLower, mass 1; collision box size=0.2 0.2 0.75; visual box size=0.2 0.2 0.75
- added link Right, mass 1; collision box size=0.75 0.2 0.2; visual box size=0.75 0.2 0.2
- added link RightLower, mass 1; collision box size=0.2 0.2 0.75; visual box size=0.2 0.2 0.75
Joints:
- added joint Left_LeftLower: type revolute, parent Left, child LeftLower, origin xyz=-0.75 0 0 rpy=0 0 0, axis 1 0 0, limit lower=-3.14159 upper=3.14159 effort=0.0 velocity=0.0
- added joint Right_RightLower: type revolute, parent Right, child RightLower, origin xyz=0.75 0 0 rpy=0 0 0, axis 1 0 0, limit lower=-3.14159 upper=3.14159 effort=0.0 velocity=0.0
- added joint Torso_Left: type revolute, parent Torso, child Left, origin xyz=-0.5 0 0.75 rpy=0 0 0, axis 0 1 0, limit lower=-3.14159 upper=3.14159 effort=0.0 velocity=0.0
- added joint Torso_Right: type revolute, parent Torso, child Right, origin xyz=0.5 0 0.75 rpy=0 0 0, axis 0 1 0, limit lower=-3.14159 upper=3.14159 effort=0.0 velocity=0.0

Commit message: increased width

File: body.urdf (robot description, URDF)
Before this commit: robot robot, 13 links, 12 joints
Links:
- link Torso: geometry collision box size=2 0.5 0.5; visual box size=2 0.5 0.5
Joints:
- joint Torso_BackLeft: origin xyz=-0.25 -0.25 0.75 rpy=0 0 0 -> xyz=-0.5 -0.25 0.75 rpy=0 0 0
- joint Torso_BackRight: origin xyz=0.25 -0.25 0.75 rpy=0 0 0 -> xyz=0.5 -0.25 0.75 rpy=0 0 0
- joint Torso_FrontLeft: origin xyz=-0.25 0.25 0.75 rpy=0 0 0 -> xyz=-0.5 0.25 0.75 rpy=0 0 0
- joint Torso_FrontRight: origin xyz=0.25 0.25 0.75 rpy=0 0 0 -> xyz=0.5 0.25 0.75 rpy=0 0 0
- joint Torso_Left: origin xyz=-0.5 0 0.75 rpy=0 0 0 -> xyz=-1.0 0 0.75 rpy=0 0 0
- joint Torso_Right: origin xyz=0.5 0 0.75 rpy=0 0 0 -> xyz=1.0 0 0.75 rpy=0 0 0

Commit message: rotated robot 90 deg

File: body.urdf (robot description, URDF)
Before this commit: robot robot, 13 links, 12 joints
Links:
- link BackLeft: geometry collision box size=0.75 0.2 0.2; visual box size=0.75 0.2 0.2
- link BackRight: geometry collision box size=0.75 0.2 0.2; visual box size=0.75 0.2 0.2
- link FrontLeft: geometry collision box size=0.75 0.2 0.2; visual box size=0.75 0.2 0.2
- link FrontRight: geometry collision box size=0.75 0.2 0.2; visual box size=0.75 0.2 0.2
- link Left: geometry collision box size=0.2 0.75 0.2; visual box size=0.2 0.75 0.2
- link Right: geometry collision box size=0.2 0.75 0.2; visual box size=0.2 0.75 0.2
- link Torso: geometry collision box size=0.5 2 0.5; visual box size=0.5 2 0.5
Joints:
- joint BackLeft_BLLower: origin xyz=0 -0.75 0 rpy=0 0 0 -> xyz=-0.75 0 0 rpy=0 0 0
- joint BackRight_BRLower: origin xyz=0 -0.75 0 rpy=0 0 0 -> xyz=0.75 0 0 rpy=0 0 0
- joint FrontLeft_FLLower: origin xyz=0 0.75 0 rpy=0 0 0 -> xyz=-0.75 0 0 rpy=0 0 0
- joint FrontRight_FRLower: origin xyz=0 0.75 0 rpy=0 0 0 -> xyz=0.75 0 0 rpy=0 0 0
- joint Left_LeftLower: origin xyz=-0.75 0 0 rpy=0 0 0 -> xyz=0 -0.75 0 rpy=0 0 0
- joint Right_RightLower: origin xyz=0.75 0 0 rpy=0 0 0 -> xyz=0 0.75 0 rpy=0 0 0
- joint Torso_BackLeft: axis 1 0 0 -> 0 1 0; origin xyz=-0.5 -0.25 0.75 rpy=0 0 0 -> xyz=-0.25 -1.9 0.75 rpy=0 0 0
- joint Torso_BackRight: axis 1 0 0 -> 0 1 0; origin xyz=0.5 -0.25 0.75 rpy=0 0 0 -> xyz=0.25 -1.9 0.75 rpy=0 0 0
- joint Torso_FrontLeft: axis 1 0 0 -> 0 1 0; origin xyz=-0.5 0.25 0.75 rpy=0 0 0 -> xyz=-0.25 -0.09999999999999998 0.75 rpy=0 0 0
- joint Torso_FrontRight: axis 1 0 0 -> 0 1 0; origin xyz=0.5 0.25 0.75 rpy=0 0 0 -> xyz=0.25 -0.09999999999999998 0.75 rpy=0 0 0
- joint Torso_Left: axis 0 1 0 -> 1 0 0; origin xyz=-1.0 0 0.75 rpy=0 0 0 -> xyz=0 -2.0 0.75 rpy=0 0 0
- joint Torso_Right: axis 0 1 0 -> 1 0 0; origin xyz=1.0 0 0.75 rpy=0 0 0 -> xyz=0 0.0 0.75 rpy=0 0 0

Commit message: pretty good!

File: body.urdf (robot description, URDF)
Before this commit: robot robot, 13 links, 12 joints
Links:
- removed link Right
- removed link RightLower
Joints:
- removed joint Right_RightLower
- removed joint Torso_Right

Commit message: tail

File: body.urdf (robot description, URDF)
Before this commit: robot robot, 11 links, 10 joints
Links:
- added link Tail, mass 1; collision box size=0.75 0.2 0.2; visual box size=0.75 0.2 0.2
Joints:
- added joint LeftLower_Tail: type revolute, parent LeftLower, child Tail, origin xyz=0 0 -0.65 rpy=0 0 0, axis 0 1 0, limit lower=-3.14159 upper=3.14159 effort=0.0 velocity=0.0

Commit message: BLOCK

File: body.urdf (robot description, URDF)
Before this commit: robot robot, 12 links, 11 joints
Links:
- removed link BLLower
- removed link BRLower
- removed link BackLeft
- removed link BackRight
- removed link FLLower
- removed link FRLower
- removed link FrontLeft
- removed link FrontRight
- removed link Left
- removed link LeftLower
- removed link Tail
- link Torso: geometry collision box size=2 2 2; visual box size=2 2 2
Joints:
- removed joint BackLeft_BLLower
- removed joint BackRight_BRLower
- removed joint FrontLeft_FLLower
- removed joint FrontRight_FRLower
- removed joint LeftLower_Tail
- removed joint Left_LeftLower
- removed joint Torso_BackLeft
- removed joint Torso_BackRight
- removed joint Torso_FrontLeft
- removed joint Torso_FrontRight
- removed joint Torso_Left

Commit message: added min max robot size

File: body.urdf (robot description, URDF)
Before this commit: robot robot, 1 links, 0 joints
Links:
- link Torso: geometry collision box size=0.5 0.5 0.5; visual box size=0.5 0.5 0.5

Commit message: trying to add colors

File: body.urdf (robot description, URDF)
Before this commit: robot robot, 1 links, 0 joints
Links:
- removed link Torso
- added link 0, mass 1; collision box size=1.4861502169570429 0.8584407621265744 1.0523009821051024; visual box size=1.4861502169570429 0.8584407621265744 1.0523009821051024
- added link 1, mass 1; collision box size=1.1388611020200912 0.8963230778769132 0.6877803225477268; visual box size=1.1388611020200912 0.8963230778769132 0.6877803225477268
- added link 2, mass 1; collision box size=1.16645296961631 1.4684852896666643 1.2014282550159572; visual box size=1.16645296961631 1.4684852896666643 1.2014282550159572
Joints:
- added joint 0_1: type revolute, parent 0, child 1, origin xyz=0 -0.4292203810632872 0.75 rpy=0 0 0, axis 1 0 0, limit lower=-3.14159 upper=3.14159 effort=0.0 velocity=0.0
- added joint 1_2: type revolute, parent 1, child 2, origin xyz=0 -0.8963230778769132 0 rpy=0 0 0, axis 0 1 0, limit lower=-3.14159 upper=3.14159 effort=0.0 velocity=0.0

Commit message: sensor colors working

File: body.urdf (robot description, URDF)
Before this commit: robot robot, 3 links, 2 joints
Links:
- added link 3, mass 1; collision box size=0.5461502319422752 1.3441708690932823 0.5221573490079146; visual box size=0.5461502319422752 1.3441708690932823 0.5221573490079146
- link 0: geometry collision box size=0.9652696173172592 0.6954605685304595 0.7207295517443372; visual box size=0.9652696173172592 0.6954605685304595 0.7207295517443372
- link 1: geometry collision box size=0.9455081159323865 1.4196888369257938 1.127589207266347; visual box size=0.9455081159323865 1.4196888369257938 1.127589207266347
- link 2: geometry collision box size=1.1459052916525136 0.7530957351280919 0.7022251485655074; visual box size=1.1459052916525136 0.7530957351280919 0.7022251485655074
Joints:
- added joint 2_3: type revolute, parent 2, child 3, origin xyz=0 -0.7530957351280919 0 rpy=0 0 0, axis 0 1 0, limit lower=-3.14159 upper=3.14159 effort=0.0 velocity=0.0
- joint 0_1: axis 1 0 0 -> 0 0 1; origin xyz=0 -0.4292203810632872 0.75 rpy=0 0 0 -> xyz=0 -0.3477302842652297 0.75 rpy=0 0 0
- joint 1_2: axis 0 1 0 -> 0 0 1; origin xyz=0 -0.8963230778769132 0 rpy=0 0 0 -> xyz=0 -1.4196888369257938 0 rpy=0 0 0
