Commit message: created synapses but sim doesnt work

File: body.urdf (robot description, URDF)
Before this commit: robot robot, 4 links, 3 joints
Links:
- removed link 3
- link 0: geometry collision box size=1.0263976631304246 0.6075803371301985 1.1679004867404852; visual box size=1.0263976631304246 0.6075803371301985 1.1679004867404852
- link 1: geometry collision box size=0.8963982657968268 1.2357073156205067 1.164996397961747; visual box size=0.8963982657968268 1.2357073156205067 1.164996397961747
- link 2: geometry collision box size=0.5835553011274247 0.735944829953145 0.8668132601571648; visual box size=0.5835553011274247 0.735944829953145 0.8668132601571648
Joints:
- removed joint 2_3
- joint 0_1: axis 0 0 1 -> 1 0 0; origin xyz=0 -0.3477302842652297 0.75 rpy=0 0 0 -> xyz=0 -0.3037901685650993 0.75 rpy=0 0 0
- joint 1_2: axis 0 0 1 -> 0 1 0; origin xyz=0 -1.4196888369257938 0 rpy=0 0 0 -> xyz=0 -1.2357073156205067 0 rpy=0 0 0

Commit message: DONE! Fixed the problem with synapses

File: body.urdf (robot description, URDF)
Before this commit: robot robot, 3 links, 2 joints
Links:
- link 0: geometry collision box size=0.31081995325433576 0.7323617698344298 0.9583565397625415; visual box size=0.31081995325433576 0.7323617698344298 0.9583565397625415
- link 1: geometry collision box size=0.8432255521394183 0.5691452127175938 0.7123561747994356; visual box size=0.8432255521394183 0.5691452127175938 0.7123561747994356
- link 2: geometry collision box size=0.8550946909357016 0.25925813574258727 0.36522955279003494; visual box size=0.8550946909357016 0.25925813574258727 0.36522955279003494
Joints:
- joint 0_1: origin xyz=0 -0.3037901685650993 0.75 rpy=0 0 0 -> xyz=0 -0.3661808849172149 0.5 rpy=0 0 0
- joint 1_2: origin xyz=0 -1.2357073156205067 0 rpy=0 0 0 -> xyz=0 -0.5691452127175938 0 rpy=0 0 0

Commit message: add 1 sensor

File: body.urdf (robot description, URDF)
Before this commit: robot robot, 3 links, 2 joints
Links:
- added link 3, mass 1; collision box size=0.2530381558644613 0.8566512503910044 0.5338234540455069; visual box size=0.2530381558644613 0.8566512503910044 0.5338234540455069
- added link 4, mass 1; collision box size=0.4014975910293347 0.29713417567915845 0.9215035263118371; visual box size=0.4014975910293347 0.29713417567915845 0.9215035263118371
- added link 5, mass 1; collision box size=0.2569256406765014 0.472764000263189 0.64226063117952; visual box size=0.2569256406765014 0.472764000263189 0.64226063117952
- link 0: geometry collision box size=0.5134615920579371 0.37654897380003494 0.8839022430843719; visual box size=0.5134615920579371 0.37654897380003494 0.8839022430843719
- link 1: geometry collision box size=0.45637360455158393 0.4617935728235771 0.3991143259274497; visual box size=0.45637360455158393 0.4617935728235771 0.3991143259274497
- link 2: geometry collision box size=0.6205692563726299 0.5518946578272718 0.8350895094008165; visual box size=0.6205692563726299 0.5518946578272718 0.8350895094008165
Joints:
- added joint 2_3: type revolute, parent 2, child 3, origin xyz=0 -0.5518946578272718 0 rpy=0 0 0, axis 1 0 0, limit lower=-3.14159 upper=3.14159 effort=0.0 velocity=0.0
- added joint 3_4: type revolute, parent 3, child 4, origin xyz=0 -0.8566512503910044 0 rpy=0 0 0, axis 1 0 0, limit lower=-3.14159 upper=3.14159 effort=0.0 velocity=0.0
- added joint 4_5: type revolute, parent 4, child 5, origin xyz=0 -0.29713417567915845 0 rpy=0 0 0, axis 0 1 0, limit lower=-3.14159 upper=3.14159 effort=0.0 velocity=0.0
- joint 0_1: axis 1 0 0 -> 0 1 0; origin xyz=0 -0.3661808849172149 0.5 rpy=0 0 0 -> xyz=0 -0.18827448690001747 0.5 rpy=0 0 0
- joint 1_2: axis 0 1 0 -> 1 0 0; origin xyz=0 -0.5691452127175938 0 rpy=0 0 0 -> xyz=0 -0.4617935728235771 0 rpy=0 0 0

Commit message: works now

File: body.urdf (robot description, URDF)
Before this commit: robot robot, 6 links, 5 joints
Links:
- removed link 3
- removed link 4
- removed link 5
- link 0: geometry collision box size=0.49365677756858795 0.5520830038980326 0.8490671709087424; visual box size=0.49365677756858795 0.5520830038980326 0.8490671709087424
- link 1: geometry collision box size=0.3122937598902342 0.5183538777918244 0.35147626662999737; visual box size=0.3122937598902342 0.5183538777918244 0.35147626662999737
- link 2: geometry collision box size=0.577777981581251 0.4490919102138419 0.34633615263162143; visual box size=0.577777981581251 0.4490919102138419 0.34633615263162143
Joints:
- removed joint 2_3
- removed joint 3_4
- removed joint 4_5
- joint 0_1: axis 0 1 0 -> 1 0 0; origin xyz=0 -0.18827448690001747 0.5 rpy=0 0 0 -> xyz=0 -0.2760415019490163 0.5 rpy=0 0 0
- joint 1_2: axis 1 0 0 -> 0 0 1; origin xyz=0 -0.4617935728235771 0 rpy=0 0 0 -> xyz=0 -0.5183538777918244 0 rpy=0 0 0

Commit message: working

File: body.urdf (robot description, URDF)
Before this commit: robot robot, 3 links, 2 joints
Links:
- added link 3, mass 1; collision box size=0.46593587188176333 0.3326323216803042 0.7293634822698054; visual box size=0.46593587188176333 0.3326323216803042 0.7293634822698054
- added link 4, mass 1; collision box size=0.6416059046783913 0.2521120471683269 0.5594380638481142; visual box size=0.6416059046783913 0.2521120471683269 0.5594380638481142
- added link 5, mass 1; collision box size=0.6158884883053892 0.793245984876152 0.5512653835485124; visual box size=0.6158884883053892 0.793245984876152 0.5512653835485124
- link 0: geometry collision box size=0.5887909243234738 0.46840665637530754 0.5137094756759092; visual box size=0.5887909243234738 0.46840665637530754 0.5137094756759092
- link 1: geometry collision box size=0.5680676818937812 0.588295418431622 0.5975858438238575; visual box size=0.5680676818937812 0.588295418431622 0.5975858438238575
- link 2: geometry collision box size=0.42043950181110745 0.46412388153014206 0.3267596433066151; visual box size=0.42043950181110745 0.46412388153014206 0.3267596433066151
Joints:
- added joint 2_3: type revolute, parent 2, child 3, origin xyz=0 -0.46412388153014206 0 rpy=0 0 0, axis 0 0 1, limit lower=-3.14159 upper=3.14159 effort=0.0 velocity=0.0
- added joint 3_4: type revolute, parent 3, child 4, origin xyz=0 -0.3326323216803042 0 rpy=0 0 0, axis 0 0 1, limit lower=-3.14159 upper=3.14159 effort=0.0 velocity=0.0
- added joint 4_5: type revolute, parent 4, child 5, origin xyz=0 -0.2521120471683269 0 rpy=0 0 0, axis 0 0 1, limit lower=-3.14159 upper=3.14159 effort=0.0 velocity=0.0
- joint 0_1: axis 1 0 0 -> 0 1 0; origin xyz=0 -0.2760415019490163 0.5 rpy=0 0 0 -> xyz=0 -0.23420332818765377 0.5 rpy=0 0 0
- joint 1_2: axis 0 0 1 -> 0 1 0; origin xyz=0 -0.5183538777918244 0 rpy=0 0 0 -> xyz=0 -0.588295418431622 0 rpy=0 0 0

Commit message: added initial values to SOLUTION

File: body.urdf (robot description, URDF)
Before this commit: robot robot, 6 links, 5 joints
Links:
- removed link 3
- removed link 4
- removed link 5
- link 0: geometry collision box size=0.43512667108898684 0.8918093264173177 0.6620868373576541; visual box size=0.43512667108898684 0.8918093264173177 0.6620868373576541
- link 1: geometry collision box size=0.7982845575201039 0.7504763404251108 0.2709566988518711; visual box size=0.7982845575201039 0.7504763404251108 0.2709566988518711
- link 2: geometry collision box size=0.7273431295582495 0.8285053155400675 0.5319127713060305; visual box size=0.7273431295582495 0.8285053155400675 0.5319127713060305
Joints:
- removed joint 2_3
- removed joint 3_4
- removed joint 4_5
- joint 0_1: axis 0 1 0 -> 1 0 0; origin xyz=0 -0.23420332818765377 0.5 rpy=0 0 0 -> xyz=0 -0.44590466320865885 0.5 rpy=0 0 0
- joint 1_2: axis 0 1 0 -> 0 0 1; origin xyz=0 -0.588295418431622 0 rpy=0 0 0 -> xyz=0 -0.7504763404251108 0 rpy=0 0 0

Commit message: connections made, joint weird

File: body.urdf (robot description, URDF)
Before this commit: robot robot, 4 links, 3 joints
Links:
- link 0: geometry collision box size=0.2618788017314734 0.6081011136874733 0.4116791042428367; visual box size=0.2618788017314734 0.6081011136874733 0.4116791042428367
- link 1: geometry collision box size=0.8377323948639859 0.28887264951841884 0.7747473525724744; visual box size=0.8377323948639859 0.28887264951841884 0.7747473525724744
- link 2: geometry collision box size=0.6197765115924936 0.9112665760842744 0.3085206598950495; visual box size=0.6197765115924936 0.9112665760842744 0.3085206598950495
- link 3: geometry collision box size=0.5371141168447652 0.850050000715464 0.36037068193542293; visual box size=0.5371141168447652 0.850050000715464 0.36037068193542293
Joints:
- removed joint 0_1
- removed joint 0_3
- removed joint 1_2
- added joint 2_3: type revolute, parent 2, child 3, origin xyz=0.3098882557962468 2.1863415771574704 3.1799145411012315 rpy=0 0 0, axis 1 0 0, limit lower=-3.14159 upper=3.14159 effort=0.0 velocity=0.0
- added joint 3_1: type revolute, parent 3, child 1, origin xyz=0.3098882557962468 0.425025000357732 3.1799145411012315 rpy=0 0 0, axis 0 1 0, limit lower=-3.14159 upper=3.14159 effort=0.0 velocity=0.0
- added joint 3_2: type revolute, parent 3, child 2, origin xyz=0.3098882557962468 1.275075001073196 3.1799145411012315 rpy=0 0 0, axis 0 1 0, limit lower=-3.14159 upper=3.14159 effort=0.0 velocity=0.0

Commit message: creating body works?

File: body.urdf (robot description, URDF)
Before this commit: robot robot, 4 links, 3 joints
Links:
- removed link 2
- removed link 3
- link 0: geometry collision box size=0.4036406342744756 0.3272777679845871 0.7061249469101343; visual box size=0.4036406342744756 0.3272777679845871 0.7061249469101343
- link 1: geometry collision box size=0.3773335699750839 0.5985926917335778 0.6217235652013511; visual box size=0.3773335699750839 0.5985926917335778 0.6217235652013511
Joints:
- removed joint 2_3
- removed joint 3_1
- removed joint 3_2
- added joint 0_1: type revolute, parent 0, child 1, origin xyz=0 0 3.353062473455067 rpy=0 0 0, axis 0 1 0, limit lower=-3.14159 upper=3.14159 effort=0.0 velocity=0.0

Commit message: added file to run

File: body.urdf (robot description, URDF)
Before this commit: robot robot, 2 links, 1 joints
Links:
- added link 2, mass 1; collision box size=0.7286733881798297 0.8216680374146507 0.6388944106512197; visual box size=0.7286733881798297 0.8216680374146507 0.6388944106512197
- added link 3, mass 1; collision box size=0.5942965422053544 0.40113348071321997 0.6304268834906088; visual box size=0.5942965422053544 0.40113348071321997 0.6304268834906088
- link 0: geometry collision box size=0.25700666678230555 0.3350362761140125 0.7475792483080763; visual box size=0.25700666678230555 0.3350362761140125 0.7475792483080763
- link 1: geometry collision box size=0.6683765433874118 0.705465148329162 0.5632690167323323; visual box size=0.6683765433874118 0.705465148329162 0.5632690167323323
Joints:
- removed joint 0_1
- added joint 2_3: type revolute, parent 2, child 3, origin xyz=0 0.41083401870732533 0.31944720532560983 rpy=0 0 0, axis 0 1 0, limit lower=-3.14159 upper=3.14159 effort=0.0 velocity=0.0
- added joint 3_1: type revolute, parent 3, child 1, origin xyz=0 0.40113348071321997 0 rpy=0 0 0, axis 0 0 1, limit lower=-3.14159 upper=3.14159 effort=0.0 velocity=0.0
- added joint 3_2: type revolute, parent 3, child 2, origin xyz=0 0.20056674035660998 0.3152134417453044 rpy=0 0 0, axis 0 0 1, limit lower=-3.14159 upper=3.14159 effort=0.0 velocity=0.0

Commit message: single sim working

File: body.urdf (robot description, URDF)
Before this commit: robot robot, 4 links, 3 joints
Links:
- added link 4, mass 1; collision box size=0.7685721315501296 0.5719107128439489 0.5913187233684801; visual box size=0.7685721315501296 0.5719107128439489 0.5913187233684801
- link 0: geometry collision box size=0.7173741534951229 0.7423372531863817 0.4074756503963227; visual box size=0.7173741534951229 0.7423372531863817 0.4074756503963227
- link 1: geometry collision box size=0.6790494387613689 0.5460964315663251 0.5556044278026447; visual box size=0.6790494387613689 0.5460964315663251 0.5556044278026447
- link 2: geometry collision box size=0.37933770921754595 0.9973793474951504 0.7371848369766855; visual box size=0.37933770921754595 0.9973793474951504 0.7371848369766855
- link 3: geometry collision box size=0.30718854975326804 0.42473628640854943 0.6195095528112657; visual box size=0.30718854975326804 0.42473628640854943 0.6195095528112657
Joints:
- removed joint 2_3
- removed joint 3_1
- removed joint 3_2
- added joint 0_1: type revolute, parent 0, child 1, origin xyz=0.35868707674756145 0 3 rpy=0 0 0, axis 0 1 0, limit lower=-3.14159 upper=3.14159 effort=0.0 velocity=0.0
- added joint 0_2: type revolute, parent 0, child 2, origin xyz=-0.35868707674756145 0 3 rpy=0 0 0, axis 1 0 0, limit lower=-3.14159 upper=3.14159 effort=0.0 velocity=0.0
- added joint 0_3: type revolute, parent 0, child 3, origin xyz=0 -0.37116862659319083 3 rpy=0 0 0, axis 0 1 0, limit lower=-3.14159 upper=3.14159 effort=0.0 velocity=0.0
- added joint 2_4: type revolute, parent 2, child 4, origin xyz=-0.18966885460877297 0 -0.36859241848834273 rpy=0 0 0, axis 1 0 0, limit lower=-3.14159 upper=3.14159 effort=0.0 velocity=0.0

Commit message: testing sensor addition

File: body.urdf (robot description, URDF)
Before this commit: robot robot, 5 links, 4 joints
Links:
- added link 5, mass 1; collision box size=0.4464615072276063 0.30822400154783264 0.5768430083731908; visual box size=0.4464615072276063 0.30822400154783264 0.5768430083731908
- link 0: geometry collision box size=0.3328660072099829 0.33381663003822526 0.8142180497281257; visual box size=0.3328660072099829 0.33381663003822526 0.8142180497281257
- link 1: geometry collision box size=0.3061819578644087 0.4926678406979071 0.8081074565476667; visual box size=0.3061819578644087 0.4926678406979071 0.8081074565476667
- link 2: geometry collision box size=0.3541527384058516 0.4832634940481756 0.36403037381886694; visual box size=0.3541527384058516 0.4832634940481756 0.36403037381886694
- link 3: geometry collision box size=0.3968496080763193 0.3073793834221679 0.7801592423661579; visual box size=0.3968496080763193 0.3073793834221679 0.7801592423661579
- link 4: geometry collision box size=0.7364892282225217 0.5789136446347745 0.7124388190039355; visual box size=0.7364892282225217 0.5789136446347745 0.7124388190039355
Joints:
- removed joint 0_3
- added joint 1_5: type revolute, parent 1, child 5, origin xyz=0.15309097893220436 0 -0.40405372827383335 rpy=0 0 0, axis 0 0 1, limit lower=-3.14159 upper=3.14159 effort=0.0 velocity=0.0
- added joint 2_3: type revolute, parent 2, child 3, origin xyz=0 -0.2416317470240878 -0.18201518690943347 rpy=0 0 0, axis 0 0 1, limit lower=-3.14159 upper=3.14159 effort=0.0 velocity=0.0
- joint 0_1: axis 0 1 0 -> 0 0 1; origin xyz=0.35868707674756145 0 3 rpy=0 0 0 -> xyz=0.16643300360499144 0 3 rpy=0 0 0
- joint 0_2: origin xyz=-0.35868707674756145 0 3 rpy=0 0 0 -> xyz=0 0 2.592890975135937 rpy=0 0 0
- joint 2_4: axis 1 0 0 -> 0 0 1; origin xyz=-0.18966885460877297 0 -0.36859241848834273 rpy=0 0 0 -> xyz=0 0.2416317470240878 -0.18201518690943347 rpy=0 0 0
